File: circuit/thermostat.sch (KiCad schematic (older format))
At the start: 13 parts

Commit message: Still in progress
Parts:
- added P2: Programming, Socket_Strips:Socket_Strip_Straight_1x06_Pitch2.54mm, symbol CONN_01X06
- added Q1, Q2: BC817-40, TO_SOT_Packages_SMD:SOT-23, symbol BC817-40
- added R10, R11, R12, R13, R14, R15, R16, R17, R3, R4, R6, R9: 2K2, Resistors_SMD:R_0805_HandSoldering, symbol R
- added R2: 56R, Resistors_SMD:R_0805_HandSoldering, symbol R
- added S1, S2: 7SEGM, symbol 7SEGM
- added SW1: UP, symbol SW_PUSH_SMALL_H
- added SW2: DOWN, symbol SW_PUSH_SMALL_H
- added U1: TRIAC, Socket_Strips:Socket_Strip_Angled_1x03_Pitch2.54mm, symbol TRIAC
- C1, C2: renamed from C?; footprint (none) -> Capacitors_SMD:C_0805_HandSoldering
- D1: renamed from D?; footprint (none) -> Diodes_ThroughHole:Diode_Bridge_15.7x15.7
- D2: renamed from D?; footprint (none) -> Diodes_SMD:D_0805
- IC1: renamed from IC?; footprint DIP20 -> Housings_DIP:DIP-20_W7.62mm
- P1: renamed from P?; footprint (none) -> Socket_Strips:Socket_Strip_Angled_1x04_Pitch2.54mm
- P3: renamed from P?; footprint (none) -> Socket_Strips:Socket_Strip_Angled_1x05_Pitch2.54mm
- R1: renamed from R?; footprint (none) -> Resistors_SMD:R_0805_HandSoldering
- R5: renamed from R?; value R -> 10K; footprint (none) -> Resistors_SMD:R_0805_HandSoldering
- R7, R8: renamed from R?; value R -> 2K2; footprint (none) -> Resistors_SMD:R_0805_HandSoldering
- U2: renamed from U?; footprint DIP-6 -> Housings_DIP:DIP-6_W7.62mm_SMD
- gave numbers to parts that had none: 1
Connections:
- net GNDREF: now also U2.2, P2.1 (P1), Q1.2 (E), Q2.2 (E), SW1.1, SW2.2
- net VCC: no longer C2.1, IC1.20 (VCC), R5.1, U3.1 (OUT)
- net at P3.2 (P2): now also C2.1, IC1.20 (VCC), R5.1, U3.1 (OUT), P2.3 (P3)
- net at P3.3 (P3): now also IC1.6 ((CKOUT/XCK/INT0)PD2); no longer IC1.14 ((PCINT2/OC0A)PB2)
- net at P3.4 (P4): now also IC1.3 ((TXD)PD1); no longer IC1.13 ((PCINT1/AIN1)PB1)
- net at P3.5 (P5): now also IC1.2 ((RXD)PD0); no longer IC1.12 ((PCINT0/AIN0)PB0)
- net at IC1.1 (PA2(~RESET~/dW)), R5.2: now also P2.2 (P2)
- net at IC1.11 ((ICP)PD6): now also R6.1
- net at IC1.15 ((PCINT3/OC1A)PB3): now also R11.1
- net at IC1.16 ((PCINT4/OC1B)PB4): now also R12.1
- net at IC1.17 ((PCINT5/MOSI/DI/SDA)PB5): now also P2.6 (P6), R13.1
- net at IC1.18 ((PCINT6/MISO/DO)PB6): now also P2.5 (P5), R14.1
- net at IC1.19 ((PCINT7/USCK/SCK/SCL)PB7): now also P2.4 (P4), R15.1
- net at IC1.5 (PA0(XTAL1)): now also R4.1
- net at IC1.7 ((INT1)PD3): now also R16.1
- net at IC1.8 ((T0)PD4): now also R17.1
- net at IC1.9 ((OC0B/T1)PD5): now also R7.1
- net at P1.4 (P4), R1.2: now also P1.2 (P2)
- net at D1.2, P1.3 (P3): now also R3.2, U1.1; no longer P1.2 (P2)
- net at P1.1 (P1): now also R2.1, U1.2
- net at U2.1: now also R4.2
- net at U2.4: now also R3.1, U1.3
- net at U2.6: now also R2.2
- net at R8.1: now also IC1.12 ((PCINT0/AIN0)PB0)
- net at R8.2: now also S1.7 (Segm_A), S2.7 (Segm_A)
- net at R7.2: now also SW2.1
- new net: IC1.13 ((PCINT1/AIN1)PB1), R9.1
- new net: IC1.14 ((PCINT2/OC0A)PB2), R10.1
- new net: R12.2, S1.1 (Segm_E), S2.1 (Segm_E)
- new net: R14.2, S1.10 (Segm_G), S2.10 (Segm_G)
- new net: R11.2, S1.2 (Segm_D), S2.2 (Segm_D)
- new net: R10.2, S1.4 (Segm_C), S2.4 (Segm_C)
- new net: R15.2, S1.5 (SegmDP), S2.5 (SegmDP)
- new net: R9.2, S1.6 (Segm_B), S2.6 (Segm_B)
- new net: Q2.3 (C), S1.8 (K)
- new net: R13.2, S1.9 (Segm_F), S2.9 (Segm_F)
- new net: Q1.3 (C), S2.8 (K)
- new net: Q1.1 (B), R16.2
- new net: Q2.1 (B), R17.2
- new net: R6.2, SW1.2
- no-connect marks 0 -> 3
Other:
- moved on the sheet: C1, C2, D1, D2, IC1, P1, P3, R1, R5, R7, R8, U2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

Commit message: Finished schematic
Parts:
- removed Q1, Q2: BC817-40, TO_SOT_Packages_SMD:SOT-23, symbol BC817-40
- removed S1, S2: 7SEGM, symbol 7SEGM
- added D10, D11, D12, D13, D3, D4, D5, D6, D7, D8, D9: LED, Socket_Strips:Socket_Strip_Straight_1x02_Pitch2.54mm, symbol LED
- added R18: 2K2, Resistors_SMD:R_0805_HandSoldering, symbol R
- SW1, SW2: footprint (none) -> custom_sw:Micro_sw_1
Connections:
- net GNDREF: now also D10.1 (K), D11.1 (K), D12.1 (K), D13.1 (K), D3.1 (K), D4.1 (K), D5.1 (K), D6.1 (K), D7.1 (K), D8.1 (K), D9.1 (K)
- net at IC1.11 ((ICP)PD6): now also R4.1; no longer R6.1
- net at IC1.4 (PA1(XTAL2)): now also R7.1
- net at IC1.5 (PA0(XTAL1)): now also R6.1; no longer R4.1
- net at IC1.9 ((OC0B/T1)PD5): now also R18.1; no longer R7.1
- net at R8.2: now also D8.2 (A)
- net at R12.2: now also D10.2 (A)
- net at R14.2: now also D11.2 (A)
- net at R11.2: now also D4.2 (A)
- net at R10.2: now also D9.2 (A)
- net at R15.2: now also D6.2 (A)
- net at R9.2: now also D3.2 (A)
- net at R13.2: now also D5.2 (A)
- net at R16.2: now also D12.2 (A)
- net at R17.2: now also D7.2 (A)
- new net: D13.2 (A), R18.2
- no-connect marks 3 -> 0
Other:
- moved on the sheet: P2, P3, R10, R11, R12, R13, R14, R15, R4, R6, R7, R8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

Commit message: More adjustments to pcb
Parts:
- D1: footprint Diodes_ThroughHole:Diode_Bridge_15.7x15.7 -> custom_smd:GREC_surface_2x2
- D2: footprint Diodes_SMD:D_0805 -> Diodes_ThroughHole:D_T-1_P5.08mm_Horizontal
- U2: footprint Housings_DIP:DIP-6_W7.62mm_SMD -> custom_smd:MOC_surface_2x3_2.5
- U3: footprint TO-92 -> Socket_Strips:Socket_Strip_Straight_1x03_Pitch2.54mm
- renumbered R7 to R4, R6 to R5, R5 to R6, R4 to R7, SW2 to SW1, SW1 to SW2
Changed lines of the file:
@@
 F 0 "D1" H 1700 1650 50  0000 C CNN
 F 1 "Diode_Bridge" H 2300 1700 50  0000 C CNN
-F 2 "Diodes_ThroughHole:Diode_Bridge_15.7x15.7" H 1950 1350 50  0001 C CNN
+F 2 "custom_smd:GREC_surface_2x2" H 1950 1350 50  0001 C CNN
 F 3 "" H 1950 1350 50  0000 C CNN
 	1    1950 1350
@@
 F 0 "D2" H 2400 1750 50  0000 C CNN
 F 1 "DZ12V" H 2400 1550 50  0000 C CNN
-F 2 "Diodes_SMD:D_0805" H 2400 1650 50  0001 C CNN
+F 2 "Diodes_ThroughHole:D_T-1_P5.08mm_Horizontal" H 2400 1650 50  0001 C CNN
 F 3 "" H 2400 1650 50  0000 C CNN
 	1    2400 1650
@@
 F 0 "U3" H 2900 1600 50  0000 C CNN
 F 1 "LM78L05ACZ" H 3100 1600 50  0000 L CNN
-F 2 "TO-92" H 3100 1500 50  0000 C CIN
+F 2 "Socket_Strips:Socket_Strip_Straight_1x03_Pitch2.54mm" H 3100 1500 50  0000 C CIN
 F 3 "" H 3100 1400 50  0000 C CNN
 	1    3100 1400
@@
 F 0 "U2" H 2150 5450 50  0000 L CNN
 F 1 "MOC3063M" H 2350 5450 50  0000 L CNN
-F 2 "Housings_DIP:DIP-6_W7.62mm_SMD" H 2150 5050 50  0000 L CIN
+F 2 "custom_smd:MOC_surface_2x3_2.5" H 2150 5050 50  0000 L CIN
 F 3 "" H 2340 5250 50  0000 L CNN
 	1    2350 5250
@@
 $EndComp
 $Comp
-L R R5
+L R R6
 U 1 1 58C13DAE
 P 3250 2100
-F 0 "R5" V 3330 2100 50  0000 C CNN
+F 0 "R6" V 3330 2100 50  0000 C CNN
 F 1 "10K" V 3250 2100 50  0000 C CNN
 F 2 "Resistors_SMD:R_0805_HandSoldering" V 3180 2100 50  0001 C CNN
@@
 $EndComp
 $Comp
-L R R7
+L R R4
 U 1 1 58C14190
 P 2550 2950
-F 0 "R7" V 2630 2950 50  0000 C CNN
+F 0 "R4" V 2630 2950 50  0000 C CNN
 F 1 "2K2" V 2550 2950 50  0000 C CNN
 F 2 "Resistors_SMD:R_0805_HandSoldering" V 2480 2950 50  0001 C CNN
@@
 $EndComp
 $Comp
-L R R6
+L R R5
 U 1 1 58C19647
 P 2550 3150
-F 0 "R6" V 2630 3150 50  0000 C CNN
+F 0 "R5" V 2630 3150 50  0000 C CNN
 F 1 "2K2" V 2550 3150 50  0000 C CNN
 F 2 "Resistors_SMD:R_0805_HandSoldering" V 2480 3150 50  0001 C CNN
@@
 $EndComp
 $Comp
-L SW_PUSH_SMALL_H SW1
+L SW_PUSH_SMALL_H SW2
 U 1 1 58C199C7
 P 2150 3150
-F 0 "SW1" H 2230 3260 50  0000 C CNN
+F 0 "SW2" H 2230 3260 50  0000 C CNN
 F 1 "UP" H 2150 3400 50  0000 C CNN
 F 2 "custom_sw:Micro_sw_1" H 2150 3350 50  0001 C CNN
@@
 $EndComp
 $Comp
-L SW_PUSH_SMALL_H SW2
+L SW_PUSH_SMALL_H SW1
 U 1 1 58C19BE5
 P 2150 2950
-F 0 "SW2" H 2230 3060 50  0000 C CNN
+F 0 "SW1" H 2230 3060 50  0000 C CNN
 F 1 "DOWN" H 2150 3200 50  0000 C CNN
 F 2 "custom_sw:Micro_sw_1" H 2150 3150 50  0001 C CNN
@@
 $EndComp
 $Comp
-L R R4
+L R R7
 U 1 1 58C1E8E6
 P 5250 4300
-F 0 "R4" V 5330 4300 50  0000 C CNN
+F 0 "R7" V 5330 4300 50  0000 C CNN
 F 1 "2K2" V 5250 4300 50  0000 C CNN
 F 2 "Resistors_SMD:R_0805_HandSoldering" V 5180 4300 50  0001 C CNN

Commit message: Corrected sch and pcb
Parts:
- removed D11, D12, D13, D6, D7: LED, Socket_Strips:Socket_Strip_Straight_1x02_Pitch2.54mm, symbol LED
- removed R14, R15, R16, R17, R18: 2K2, Resistors_SMD:R_0805_HandSoldering, symbol R
- renumbered D8 to D6, D9 to D7, D10 to D8, R11 to R10, R12 to R11, R13 to R12, R5 to R13, R6 to R4, R7 to R5, R4 to R6, R8 to R7, R9 to R8, R10 to R9
Connections:
- net at P3.3 (P3): now also IC1.8 ((T0)PD4); no longer IC1.6 ((CKOUT/XCK/INT0)PD2)
- net at P3.4 (P4): now also IC1.7 ((INT1)PD3); no longer IC1.3 ((TXD)PD1)
- net at P3.5 (P5): now also IC1.6 ((CKOUT/XCK/INT0)PD2); no longer IC1.2 ((RXD)PD0)
- net at IC1.12 ((PCINT0/AIN0)PB0): now also R6.1; no longer R7.1
- net at IC1.13 ((PCINT1/AIN1)PB1): now also R7.1; no longer R8.1
- net at IC1.14 ((PCINT2/OC0A)PB2): now also R8.1; no longer R9.1
- net at IC1.15 ((PCINT3/OC1A)PB3): now also R9.1; no longer R10.1
- net at IC1.16 ((PCINT4/OC1B)PB4): now also R10.1; no longer R11.1
- net at IC1.17 ((PCINT5/MOSI/DI/SDA)PB5), P2.6 (P6): now also R11.1; no longer R12.1
- net at IC1.18 ((PCINT6/MISO/DO)PB6), P2.5 (P5): now also R12.1
- net at IC1.19 ((PCINT7/USCK/SCK/SCL)PB7), P2.4 (P4): now also R13.1
- net at IC1.4 (PA1(XTAL2)): no longer R6.1
- net at IC1.5 (PA0(XTAL1)): no longer R13.1
- no-connect marks 0 -> 5
Other:
- moved on the sheet: D3, D4, D5, D6, D7, D8, R10, R11, R12, R13, R6, R7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

Commit message: Finished the FW
Parts:
- added P4: UART TX, Socket_Strips:Socket_Strip_Straight_1x01_Pitch2.54mm, symbol CONN_01X01
- R1: footprint Resistors_SMD:R_0805_HandSoldering -> Resistors_ThroughHole:R_Axial_DIN0204_L3.6mm_D1.6mm_P7.62mm_Horizontal
Connections:
- net at P3.3 (P3): now also IC1.7 ((INT1)PD3); no longer IC1.8 ((T0)PD4)
- net at P3.4 (P4): now also IC1.8 ((T0)PD4); no longer IC1.7 ((INT1)PD3)
- net at P3.5 (P5): now also IC1.9 ((OC0B/T1)PD5); no longer IC1.6 ((CKOUT/XCK/INT0)PD2)
- net at IC1.11 ((ICP)PD6): no longer R5.1
- net at IC1.3 ((TXD)PD1): now also P4.1 (P1)
- new net: IC1.6 ((CKOUT/XCK/INT0)PD2), R5.1
- no-connect marks 5 -> 4
Other:
- moved on the sheet: R5
Changed lines of the file:
@@
 F 0 "R1" V 1400 1000 50  0000 C CNN
 F 1 "R" V 1500 950 50  0000 C CNN
-F 2 "Resistors_SMD:R_0805_HandSoldering" V 1430 950 50  0001 C CNN
+F 2 "Resistors_ThroughHole:R_Axial_DIN0204_L3.6mm_D1.6mm_P7.62mm_Horizontal" V 1430 950 50  0001 C CNN
 F 3 "" H 1500 950 50  0000 C CNN
 	1    1500 950
@@
 $EndComp
 $Comp
-L GNDREF #PWR1
+L GNDREF #PWR01
 U 1 1 58C13B33
 P 3950 5750
-F 0 "#PWR1" H 3950 5500 50  0001 C CNN
+F 0 "#PWR01" H 3950 5500 50  0001 C CNN
 F 1 "GNDREF" H 3950 5600 50  0000 C CNN
 F 2 "" H 3950 5750 50  0000 C CNN
@@
 L R R5
 U 1 1 58C1E8E6
-P 5250 4300
-F 0 "R5" V 5330 4300 50  0000 C CNN
-F 1 "2K2" V 5250 4300 50  0000 C CNN
-F 2 "Resistors_SMD:R_0805_HandSoldering" V 5180 4300 50  0001 C CNN
-F 3 "" H 5250 4300 50  0000 C CNN
-	1    5250 4300
+P 5300 4850
+F 0 "R5" V 5380 4850 50  0000 C CNN
+F 1 "2K2" V 5300 4850 50  0000 C CNN
+F 2 "Resistors_SMD:R_0805_HandSoldering" V 5230 4850 50  0001 C CNN
+F 3 "" H 5300 4850 50  0000 C CNN
+	1    5300 4850
 	1    0    0    -1
 $EndComp
@@
 $EndComp
 $Comp
-L GNDREF #PWR2
+L GNDREF #PWR02
 U 1 1 58C18559
 P 6100 1950
-F 0 "#PWR2" H 6100 1700 50  0001 C CNN
+F 0 "#PWR02" H 6100 1700 50  0001 C CNN
 F 1 "GNDREF" H 6100 1800 50  0000 C CNN
 F 2 "" H 6100 1950 50  0000 C CNN
@@
 	-1   0    0    1
 $EndComp
+NoConn ~ 2800 2950
+NoConn ~ 2800 3150
+NoConn ~ 5100 3550
 Wire Wire Line
 	5100 3250 7600 3250
@@
 	5100 2650 7600 2650
 Wire Wire Line
-	5900 1250 5900 3950
-Wire Wire Line
-	5800 1250 5800 3850
-Wire Wire Line
-	5700 1250 5700 3750
+	5800 1250 5800 3950
+Wire Wire Line
+	5700 1250 5700 4050
 Wire Wire Line
 	2350 1350 2700 1350
@@
 	6100 1250 6100 1950
 Wire Wire Line
-	5100 4150 5250 4150
-Wire Wire Line
 	2650 2100 2650 2650
 Wire Wire Line
@@
 	2400 1850 2400 1900
 Wire Wire Line
-	2650 5150 5250 5150
-Wire Wire Line
-	5250 5150 5250 4450
+	2650 5150 5300 5150
 Wire Wire Line
 	2650 5700 3950 5700
 Wire Wire Line
 	8650 1900 8650 3350
-Wire Wire Line
-	5700 3750 5100 3750
-Wire Wire Line
-	5800 3850 5100 3850
-Wire Wire Line
-	5900 3950 5100 3950
 Wire Wire Line
 	8300 2650 8650 2650
@@
 	8650 3350 8300 3350
 Connection ~ 8650 3250
-NoConn ~ 2800 2950
-NoConn ~ 2800 3150
-NoConn ~ 5100 3550
-NoConn ~ 5100 3650
-NoConn ~ 5100 4050
+Wire Wire Line
+	5300 5150 5300 5000
+Wire Wire Line
+	5300 4700 5300 3750
+Wire Wire Line
+	5300 3750 5100 3750
+Wire Wire Line
+	5900 1250 5900 3850
+Wire Wire Line
+	5700 4050 5100 4050
+Wire Wire Line
+	5800 3950 5100 3950
+Wire Wire Line
+	5900 3850 5100 3850
+NoConn ~ 5100 4150
+$Comp
+L CONN_01X01 P4
+U 1 1 58C273E5
+P 5450 3650
+F 0 "P4" H 5450 3750 50  0000 C CNN
+F 1 "UART TX" H 5500 3550 50  0000 C CNN
+F 2 "Socket_Strips:Socket_Strip_Straight_1x01_Pitch2.54mm" H 5450 3650 50  0001 C CNN
+F 3 "" H 5450 3650 50  0000 C CNN
+	1    5450 3650
+	1    0    0    -1
+$EndComp
+Wire Wire Line
+	5250 3650 5100 3650
 $EndSCHEMATC
