File: circuit/thermostat.kicad_pcb (KiCad board)
At the start: 2 copper layers, 41 parts, among them IC1 ATTINY2313-P, P1 PWR+HEATER, P2 Programming, P3 MODULE, SW1 UP, SW2 DOWN, U1 TRIAC, U2 MOC3063M

Commit message: More adjustments to pcb
Parts:
- added U3: LM78L05ACZ, Socket_Strips:Socket_Strip_Straight_1x03_Pitch2.54mm, F.Cu at (168.9, 29.2)
- D1: footprint Diodes_ThroughHole:Diode_Bridge_15.7x15.7 -> custom_smd:GREC_surface_2x2
- D2: footprint Diodes_SMD:D_0805 -> Diodes_ThroughHole:D_T-1_P5.08mm_Horizontal
- R5: value 10K -> 2K2
- R6: value 2K2 -> 10K
- SW1: value UP -> DOWN
- SW2: value DOWN -> UP
- U2: footprint Housings_DIP:DIP-6_W7.62mm_SMD -> custom_smd:MOC_surface_2x3_2.5
- moved SW1 182.6 mm to (59.5, 135.6)
- moved U1 182.6 mm to (54.3, 134.1)
- moved D2 165.2 mm to (96.5, 161.3), turned to 180 degrees
- moved R6 129.3 mm to (108.0, 95.2)
- moved D12 128.6 mm to (160.0, 153.7), turned to 270 degrees
- moved D13 122.1 mm to (160.0, 143.5), turned to 270 degrees
- moved R18 121.6 mm to (152.4, 143.5)
- moved R11 114.9 mm to (152.4, 123.2)
- moved D3 109.7 mm to (160.0, 133.3), turned to 270 degrees
- moved D8 104.2 mm to (160.0, 138.4), turned to 270 degrees
- moved R14 101.7 mm to (152.4, 108.0)
- moved R17 100.9 mm to (152.4, 148.6)
- moved R5 99.3 mm to (125.7, 95.2)
- moved R16 98.7 mm to (152.4, 153.7)
- moved R7 93.4 mm to (139.7, 96.5)
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Connections:
- R4 pad 1: Net-(IC1-Pad11) -> Net-(IC1-Pad4)
- R5 pad 1: Net-(C2-Pad1) -> Net-(IC1-Pad5)
- R5 pad 2: Net-(IC1-Pad1) -> Net-(R5-Pad2)
- R6 pad 1: Net-(IC1-Pad5) -> Net-(C2-Pad1)
- R6 pad 2: Net-(R6-Pad2) -> Net-(IC1-Pad1)
- R7 pad 1: Net-(IC1-Pad4) -> Net-(IC1-Pad11)
- SW1 pad 1: GNDREF -> Net-(R4-Pad2)
- SW1 pad 2: Net-(R6-Pad2) -> GNDREF
- SW2 pad 1: Net-(R7-Pad2) -> GNDREF
- SW2 pad 2: GNDREF -> Net-(R5-Pad2)
- U2 pad 1: Net-(R4-Pad2) -> Net-(R7-Pad2)
Routing:
- net (no net): track 0.00 -> 204.5 mm
- net Net-(IC1-Pad15): track 0.00 -> 10.1 mm

Commit message: Corrected sch and pcb
Parts:
- removed D10, D11, D12, D13, D9: LED, Socket_Strips:Socket_Strip_Straight_1x02_Pitch2.54mm
- removed R14, R15, R16, R17, R18: 2K2, Resistors_SMD:R_0805_HandSoldering
- R4: value 2K2 -> 10K
- R6: value 10K -> 2K2
- moved P3 114.3 mm to (87.6, 123.2)
- moved SW1 99.5 mm to (158.8, 143.5), turned to 90 degrees
- moved U2 99.1 mm to (102.9, 149.9)
- moved P2 82.8 mm to (144.8, 108.0)
- moved U3 80.7 mm to (142.2, 105.4), turned to 90 degrees
- moved P1 80.0 mm to (128.3, 92.7), turned to 270 degrees
- moved R4 73.2 mm to (138.4, 113.0), turned to 180 degrees
- moved R6 66.5 mm to (153.7, 143.5)
- moved D1 63.7 mm to (142.2, 97.8), turned to 270 degrees
- moved R1 56.5 mm to (141.0, 85.1)
- moved R3 53.4 mm to (120.7, 127.0)
- moved R5 52.8 mm to (116.8, 147.3)
- moved R2 50.1 mm to (119.4, 120.7)
- moved C2 48.2 mm to (142.2, 108.0)
- moved R7 45.0 mm to (156.2, 138.4)
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Connections:
- P3 pad 3: Net-(IC1-Pad6) -> Net-(IC1-Pad8)
- P3 pad 4: Net-(IC1-Pad3) -> Net-(IC1-Pad7)
- P3 pad 5: Net-(IC1-Pad2) -> Net-(IC1-Pad6)
- R10 pad 1: Net-(IC1-Pad14) -> Net-(IC1-Pad16)
- R10 pad 2: Net-(D9-Pad2) -> Net-(D4-Pad2)
- R11 pad 1: Net-(IC1-Pad15) -> Net-(IC1-Pad17)
- R11 pad 2: Net-(D4-Pad2) -> Net-(D8-Pad2)
- R12 pad 1: Net-(IC1-Pad16) -> Net-(IC1-Pad18)
- R12 pad 2: Net-(D10-Pad2) -> Net-(D5-Pad2)
- R13 pad 1: Net-(IC1-Pad17) -> Net-(IC1-Pad19)
- R13 pad 2: Net-(D5-Pad2) -> Net-(R13-Pad2)
- R4 pad 1: Net-(IC1-Pad4) -> Net-(C2-Pad1)
- R4 pad 2: Net-(R4-Pad2) -> Net-(IC1-Pad1)
- R5 pad 1: Net-(IC1-Pad5) -> Net-(IC1-Pad11)
- R6 pad 1: Net-(C2-Pad1) -> Net-(IC1-Pad12)
- R6 pad 2: Net-(IC1-Pad1) -> Net-(R6-Pad2)
- R7 pad 1: Net-(IC1-Pad11) -> Net-(IC1-Pad13)
- R7 pad 2: Net-(R7-Pad2) -> Net-(D6-Pad2)
- R8 pad 1: Net-(IC1-Pad12) -> Net-(IC1-Pad14)
- R8 pad 2: Net-(D8-Pad2) -> Net-(D3-Pad2)
- R9 pad 1: Net-(IC1-Pad13) -> Net-(IC1-Pad15)
- R9 pad 2: Net-(D3-Pad2) -> Net-(D7-Pad2)
- SW1 pad 1: Net-(R4-Pad2) -> Net-(R6-Pad2)
- SW2 pad 2: Net-(R5-Pad2) -> Net-(R13-Pad2)
- U2 pad 1: Net-(R7-Pad2) -> Net-(R5-Pad2)
Routing:
- net (no net): track 204.5 -> 0.00 mm
- net GNDREF: track 0.00 -> 135.9 mm, vias 0 -> 1
- net Net-(IC1-Pad13): track 0.00 -> 20.2 mm
- net Net-(IC1-Pad12): track 0.00 -> 20.2 mm
- net Net-(IC1-Pad18): track 0.00 -> 17.7 mm
- net Net-(IC1-Pad14): track 0.00 -> 17.7 mm
- net Net-(IC1-Pad19): track 0.00 -> 17.7 mm
- net Net-(C2-Pad1): track 0.00 -> 16.5 mm
- net Net-(IC1-Pad1): track 0.00 -> 15.2 mm, vias 0 -> 2
- net Net-(IC1-Pad17): track 0.00 -> 15.1 mm
- net Net-(IC1-Pad16): track 0.00 -> 12.6 mm
- net Net-(R6-Pad2): track 0.00 -> 10.2 mm
- net Net-(R13-Pad2): track 0.00 -> 10.2 mm
- net Net-(C1-Pad1): track 0.00 -> 5.08 mm, vias 0 -> 1
- net Net-(IC1-Pad15): track 10.1 -> 15.1 mm

Commit message: Finished the FW
Parts:
- added P4: UART TX, Socket_Strips:Socket_Strip_Straight_1x01_Pitch2.54mm, F.Cu at (132.1, 118.1)
- R1: footprint Resistors_SMD:R_0805_HandSoldering -> Resistors_ThroughHole:R_Axial_DIN0204_L3.6mm_D1.6mm_P7.62mm_Horizontal
- moved U1 50.4 mm to (127.0, 115.6), turned to 270 degrees
- moved D2 41.2 mm to (149.9, 100.3), turned to 90 degrees
- moved P3 37.5 mm to (121.9, 138.4), turned to 90 degrees
- moved U2 34.3 mm to (124.5, 123.2), turned to 90 degrees
- moved R5 26.4 mm to (132.1, 125.7), turned to 180 degrees
- moved R1 12.0 mm to (134.6, 95.2), turned to 270 degrees
- moved R2 10.9 mm to (123.2, 110.5), turned to 180 degrees
- moved R3 9.67 mm to (124.5, 118.1)
- moved P1 2.84 mm to (129.5, 95.2), turned to 0 degrees
Connections:
- IC1 pad 11: Net-(IC1-Pad11) -> (no net)
- IC1 pad 2: Net-(IC1-Pad2) -> (no net)
- IC1 pad 4: Net-(IC1-Pad4) -> (no net)
- IC1 pad 5: Net-(IC1-Pad5) -> (no net)
- P3 pad 3: Net-(IC1-Pad8) -> Net-(IC1-Pad7)
- P3 pad 4: Net-(IC1-Pad7) -> Net-(IC1-Pad8)
- P3 pad 5: Net-(IC1-Pad6) -> Net-(IC1-Pad9)
- R5 pad 1: Net-(IC1-Pad11) -> Net-(IC1-Pad6)
Routing:
- net GNDREF: track 135.9 -> 195.6 mm, vias 1 -> 3
- net Net-(C2-Pad1): track 16.5 -> 62.3 mm
- net Net-(D1-Pad2): track 0.00 -> 31.7 mm, vias 0 -> 2
- net Net-(P1-Pad1): track 0.00 -> 30.5 mm
- net Net-(R2-Pad2): track 0.00 -> 24.1 mm
- net Net-(IC1-Pad7): track 0.00 -> 17.8 mm
- net Net-(P1-Pad2): track 0.00 -> 15.2 mm
- net Net-(IC1-Pad8): track 0.00 -> 12.7 mm
- net Net-(C1-Pad1): track 5.08 -> 16.5 mm, vias 1 -> 2
- net Net-(IC1-Pad9): track 0.00 -> 7.62 mm
- net Net-(R3-Pad1): track 0.00 -> 7.54 mm
- net Net-(IC1-Pad3): track 0.00 -> 2.54 mm
- net Net-(D1-Pad4): track 0.00 -> 2.54 mm
- net Net-(R5-Pad2): track 0.00 -> 1.19 mm
- net Net-(IC1-Pad6): track 0.00 -> 1.19 mm

Commit message: PCB reduced
Parts:
- moved R7 14.8 mm to (143.5, 130.8)
- moved R6 14.4 mm to (143.5, 133.3)
- moved R8 13.7 mm to (143.5, 128.3)
- moved R9 13.0 mm to (143.5, 125.7)
- moved R10 12.7 mm to (143.5, 123.2)
- moved R12 11.4 mm to (146.1, 118.1)
- moved R13 10.8 mm to (146.1, 115.6)
- moved R11 10.5 mm to (146.1, 120.7)
- moved D4 3.59 mm to (157.5, 125.7)
- moved D8 3.59 mm to (157.5, 120.7)
- moved D3 3.59 mm to (157.5, 135.9)
- moved D5 3.59 mm to (157.5, 115.6)
- moved D6 3.59 mm to (157.5, 141.0)
- moved D7 3.59 mm to (157.5, 130.8)
- moved SW1 3.59 mm to (156.2, 146.1), turned to 270 degrees
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Routing:
- net Net-(IC1-Pad13): track 20.2 -> 0.00 mm
- net Net-(IC1-Pad12): track 20.2 -> 0.00 mm
- net Net-(D6-Pad2): track 0.00 -> 20.2 mm
- net Net-(IC1-Pad14): track 17.7 -> 0.00 mm
- net Net-(D3-Pad2): track 0.00 -> 17.7 mm
- net Net-(IC1-Pad18): track 17.7 -> 2.54 mm
- net Net-(IC1-Pad19): track 17.7 -> 2.54 mm
- net Net-(D7-Pad2): track 0.00 -> 15.2 mm
- net Net-(IC1-Pad15): track 15.1 -> 0.00 mm
- net Net-(R6-Pad2): track 10.2 -> 25.3 mm
- net Net-(IC1-Pad16): track 12.6 -> 0.00 mm
- net Net-(D4-Pad2): track 0.00 -> 12.6 mm
- net Net-(IC1-Pad17): track 15.1 -> 2.54 mm
- net GNDREF: track 195.6 -> 185.5 mm, vias 3 -> 2
- net Net-(D5-Pad2): track 0.00 -> 10.1 mm
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